Commit message: Add optical-axis board follow with HUD start, handeye, and stow.
Keep the CDC bridge holding torque while homing, reject bad PnP jumps, and require stow before any limp restart.

Co-authored-by: Cursor <cursoragent@cursor.com>

File: dummy_moveit_ws/dummy-ros2_description/urdf/dummy.urdf (robot description, URDF)
Before this commit: robot dummy-ros2, 8 links, 7 joints
Joints:
- joint Joint2: limit lower=-1.308997 upper=1.570796 effort=150 velocity=3.15 -> lower=-2.094395 upper=1.745329 effort=150 velocity=3.15
- joint Joint3: limit lower=-1.570796 upper=1.570796 effort=150 velocity=3.15 -> lower=-2.617994 upper=2.617994 effort=150 velocity=3.15
