Commit message: Stabilize optical board follow: stream CDC, lock J4/J6, and start at [0,0,90,0,0,0].
Translation-only servo was winding J4 ~180° and slamming J5/J1 into software walls; the bridge now clips per-axis, holds roll joints at follow-start, and goto waits for firmware instead of jerky hops.

Co-authored-by: Cursor <cursoragent@cursor.com>

File: dummy_moveit_ws/dummy-ros2_description/urdf/dummy-ros2.xacro (robot description, xacro)
@@ -155,7 +155,8 @@
   <child link="link1_1_1"/>
   <axis xyz="0.0 0.0 1.0"/>
-  <limit
-    lower="-3.141593"
-    upper="3.141593"
+  <!-- URDF = hardware range. CDC bridge keeps a 1.5° bumper (joint_limits_fw.py). -->
+  <limit
+    lower="-3.14159"
+    upper="3.14159"
     effort="150"
     velocity="3.15"/>
@@ -167,6 +168,6 @@
   <axis xyz="1.0 0.0 -0.0"/>
   <limit
-    lower="-1.308997"
-    upper="1.570796"
+    lower="-2.09440"
+    upper="1.74533"
     effort="150"
     velocity="3.15" />
@@ -178,6 +179,6 @@
   <axis xyz="1.0 -0.0 -0.0"/>
   <limit
-    lower="-1.570796"
-    upper="1.570796"
+    lower="-2.61799"
+    upper="2.61799"
     effort="150"
     velocity="3.15" />
@@ -189,6 +190,6 @@
   <axis xyz="0.0 -1.0 0.0"/>
   <limit
-    lower="-3.14"
-    upper="3.14"
+    lower="-3.14159"
+    upper="3.14159"
     effort="150"
     velocity="3.15" />
@@ -200,6 +201,6 @@
   <axis xyz="-1.0 -0.0 0.0"/>
   <limit
-    lower="-1.570796"
-    upper="1.570796"
+    lower="-1.57080"
+    upper="1.57080"
     effort="150"
     velocity="3.15" />
@@ -211,6 +212,6 @@
   <axis xyz="0.0 1.0 -0.0"/>
   <limit
-    lower="-3.14"
-    upper="3.14"
+    lower="-3.14159"
+    upper="3.14159"
     effort="150"
     velocity="3.15" />

File: dummy_moveit_ws/dummy-ros2_description/urdf/dummy.urdf (robot description, URDF)
Before this commit: robot dummy-ros2, 8 links, 7 joints
Joints:
- joint Joint1: limit lower=-3.141593 upper=3.141593 effort=150 velocity=3.15 -> lower=-3.14159 upper=3.14159 effort=150 velocity=3.15
- joint Joint2: limit lower=-2.094395 upper=1.745329 effort=150 velocity=3.15 -> lower=-2.09440 upper=1.74533 effort=150 velocity=3.15
- joint Joint3: limit lower=-2.617994 upper=2.617994 effort=150 velocity=3.15 -> lower=-2.61799 upper=2.61799 effort=150 velocity=3.15
- joint Joint4: limit lower=-3.14 upper=3.14 effort=150 velocity=3.15 -> lower=-3.14159 upper=3.14159 effort=150 velocity=3.15
- joint Joint5: limit lower=-1.570796 upper=1.570796 effort=150 velocity=3.15 -> lower=-1.57080 upper=1.57080 effort=150 velocity=3.15
- joint Joint6: limit lower=-3.14 upper=3.14 effort=150 velocity=3.15 -> lower=-3.14159 upper=3.14159 effort=150 velocity=3.15
